File: rPi_audio_board_V0.4.sch (KiCad schematic (older format))
At the start: 50 parts, among them J1 RASPI_IO_HEADER, J2 CONN_4X2, J3 PIN OUT, P1 9V DC, P2 Headphone Out, P3 CONNECTOR_3, P4 CONNECTOR_3, P5 MODE SET, P6 CONNECTOR_3, U1 MIC5207BM5, U2 MIC39100-5.0, U3 MIC5225, U4 TLE2426, U5 WM8731, U6 DRV135, U7 DRV135, X1 12.288MHz

Commit message: better file labelling
Other:
- note added: "A header breakout for debugging \nand analysis of digital signals.\nNot implemented on first boards"
- note removed: "A header breakout for debugging \nand analysis of digital signals"
Changed lines of the file:
@@
 EESchema Schematic File Version 2
+LIBS:w_vacuum
+LIBS:device
+LIBS:power
+LIBS:w_analog
+LIBS:w_connectors
+LIBS:w_device
+LIBS:w_logic
+LIBS:w_memory
+LIBS:w_microcontrollers
+LIBS:w_opto
+LIBS:w_relay
+LIBS:w_rtx
+LIBS:w_transistor
 LIBS:rPi_audio_board_4-cache
+LIBS:rPi_audio_board_V0.4-cache
 EELAYER 24 0
 EELAYER END
@@
 Text GLabel 6500 1600 2    60   Output ~ 0
 DVDD
-Text Notes 4750 1350 0    60   ~ 0
+Text Notes 4650 1250 0    60   ~ 0
 Check pin orientation\n because P5 is mounted upside down!
 $Comp
@@
 Wire Wire Line
 	1300 1500 1450 1500
-Text Notes 7450 1300 0    60   ~ 0
-A header breakout for debugging \nand analysis of digital signals
+Text Notes 7350 1100 0    60   ~ 0
+A header breakout for debugging \nand analysis of digital signals.\nNot implemented on first boards
 Text Notes 12500 4450 0    60   ~ 0
 This crystal can be replaced eventually\nwith a programmable PLL clock
@@
 	3250 1400 3050 1400
 Connection ~ 2050 10300
-Text Notes 3500 9250 0    60   ~ 0
+Text Notes 3000 8500 0    60   ~ 0
 SMd poarts sizes: 0805 seems standard for resistors. Try this for caps too and inductors if possible.\n
 $Comp
