File: rPi_audio_board_V0.8.sch (KiCad schematic (older format))
At the start: 52 parts, among them J1 RASPI_IO_HEADER, J2 CONN_4X2, J3 PIN OUT, P1 9V DC, P2 Headphone Out, P3 CONNECTOR_3, P4 CONNECTOR_3, P5 MODE SET, P6 CONNECTOR_3, U1 MIC5207BM5, U2 MIC39100-5.0, U3 MIC5225, U4 TLE2426, U5 WM8731, U6 DRV135, U7 DRV135, X1 12.288MHz

Commit message: board revised design
Parts:
- removed C8, C9: 220uF, symbol CP1
- removed P2: Headphone Out, symbol CONNECTOR_3
- removed P4: CONNECTOR_3, symbol CONNECTOR_3
- added C20, C21: 1uF, symbol CP1
- added C8, C9: 220pF, symbol C
- added C? (x2): 1uF, symbol C
- added C?: 47uf, symbol CP1
- added D?: 3v zener, symbol ZENER
- added J4: Power, symbol HEADER_2X2
- added J5: Line IN, symbol HEADER_3
- added J6: Unbal L, symbol HEADER_2
- added J7: Unbal R, symbol HEADER_2
- added LD1: Red, symbol LED
- added LD2, LD3, LD4, LD5: Green, symbol LED
- added R13: 3k6, symbol R
- added R14: 1k6, symbol R
- added R15, R17: 750, symbol R
- added R16: 3k9, symbol R
- added R18, R19: 5k6, symbol R
- added R? (x2): 47k, symbol R
- C15: value 10uF -> 47uF
- P3: value CONNECTOR_3 -> Bal L
- P6: value CONNECTOR_3 -> Bal R
- R3, R4: value 10k -> 5k6
- gave numbers to parts that had none: 2
Connections:
- net labels added: INL, INR
- net labels removed: GNDPWR, GPIO15, LHPOUT, RHPOUT
- wire segments 177 -> 199
- no-connect marks 3 -> 22
Other:
- note added: "\n\n\n"
- note removed: "Diode protection for SMD LDO's\n\nSeries poly fuse and shunt bi-directional junction MOV \n\nJumper for disconnecting 5v supply to rPi\n\nPolarity protection - series low Fv drop diode?"
- note removed: "These caps are SMD electrolytic cans. 10mm?"
- moved on the sheet: P1
